Commit message: Include mass/inertia properties in Panda URDFs

File: franka_description/robots/common/hand.xacro (robot description, xacro)
@@ -1,6 +1,27 @@
 <?xml version="1.0" encoding="utf-8"?>
 <robot xmlns:xacro="http://www.ros.org/wiki/xacro" name="hand">
+  <!-- ============================================================== -->
+  <!-- Macro to add an <inertial> tag based on yaml-load properties   -->
+  <!--                                                                -->
+  <!-- name:     Name of the end_effector (without prefix)              -->
+  <!-- ee_inertials: Dictionary of inertia properties (see inertial.yaml) -->
+  <!-- ============================================================== -->
+  <xacro:macro name="ee-inertials" params="name ee_inertials:=^">
+      <xacro:unless value="${name in ee_inertials}">${xacro.warning('No inertia properties defined for: ' + name)}</xacro:unless>
+      <xacro:if value="${name in ee_inertials}">
+        <!-- Access inertia properties of link 'name' -->
+        <xacro:property name="link_inertials" value="${ee_inertials[name]}" lazy_eval="false" />
+        <inertial>
+          <origin rpy="${link_inertials.origin.rpy}" xyz="${link_inertials.origin.xyz}" />
+          <mass value="${link_inertials.mass}" />
+          <xacro:if value="${'inertia' in link_inertials}">
+            <xacro:property name="I" value="${link_inertials.inertia}" />
+            <inertia ixx="${I.xx}" ixy="${I.xy}" ixz="${I.xz}" iyy="${I.yy}" iyz="${I.yz}" izz="${I.zz}" />
+          </xacro:if>
+        </inertial>
+      </xacro:if>
+  </xacro:macro>
   <!-- safety_distance: Minimum safety distance in [m] by which the collision volumes are expanded and which is enforced during robot motions -->
-  <xacro:macro name="hand" params="connected_to:='' ns:='' rpy:='0 0 0' xyz:='0 0 0' safety_distance:=0">
+  <xacro:macro name="hand" params="connected_to:='' ns:='' rpy:='0 0 0' xyz:='0 0 0' safety_distance:=0 ee_inertials:=^">
     <xacro:unless value="${connected_to == ''}">
       <joint name="${ns}_hand_joint" type="fixed">
@@ -52,4 +73,5 @@
         </geometry>
       </collision>
+      <xacro:ee-inertials name="${ns}_hand" />
     </link>
     <!-- Define the hand_tcp frame -->
@@ -94,4 +116,5 @@
         </geometry>
       </collision>
+      <xacro:ee-inertials name="${ns}_leftfinger" />
     </link>
     <link name="${ns}_rightfinger">
@@ -130,4 +153,5 @@
         </geometry>
       </collision>
+      <xacro:ee-inertials name="${ns}_rightfinger" />
     </link>
     <joint name="${ns}_finger_joint1" type="prismatic">

File: franka_description/robots/common/panda_arm.xacro (robot description, xacro)
@@ -1,7 +1,28 @@
 <?xml version='1.0' encoding='utf-8'?>
 <robot xmlns:xacro="http://www.ros.org/wiki/xacro" name="panda">
+  <!-- ============================================================== -->
+  <!-- Macro to add an <inertial> tag based on yaml-load properties   -->
+  <!--                                                                -->
+  <!-- name:     Name of the robot link (without prefix)              -->
+  <!-- inertial: Dictionary of inertia properties (see inertial.yaml) -->
+  <!-- ============================================================== -->
+  <xacro:macro name="panda-inertials" params="name inertials:=^">
+      <xacro:unless value="${name in inertials}">${xacro.warning('No inertia properties defined for: ' + name)}</xacro:unless>
+      <xacro:if value="${name in inertials}">
+        <!-- Access inertia properties of link 'name' -->
+        <xacro:property name="link_inertials" value="${inertials[name]}" lazy_eval="false" />
+        <inertial>
+          <origin rpy="${link_inertials.origin.rpy}" xyz="${link_inertials.origin.xyz}" />
+          <mass value="${link_inertials.mass}" />
+          <xacro:if value="${'inertia' in link_inertials}">
+            <xacro:property name="I" value="${link_inertials.inertia}" />
+            <inertia ixx="${I.xx}" ixy="${I.xy}" ixz="${I.xz}" iyy="${I.yy}" iyz="${I.yz}" izz="${I.zz}" />
+          </xacro:if>
+        </inertial>
+      </xacro:if>
+  </xacro:macro>
   <!-- safety_distance: Minimum safety distance in [m] by which the collision volumes are expanded and which is enforced during robot motions -->
   <!-- arm_id: Namespace of the panda arm. Serves to differentiate between arms in case of multiple instances. -->
-  <xacro:macro name="panda_arm" params="arm_id:='panda' description_pkg:='franka_description' connected_to:='' xyz:='0 0 0' rpy:='0 0 0' safety_distance:=0">
+  <xacro:macro name="panda_arm" params="arm_id:='panda' description_pkg:='franka_description' connected_to:='' xyz:='0 0 0' rpy:='0 0 0' safety_distance:=0 inertials=^">
     <xacro:unless value="${not connected_to}">
       <joint name="${arm_id}_joint_${connected_to}" type="fixed">
@@ -35,4 +56,5 @@
         </geometry>
       </collision>
+      <xacro:panda-inertials name="${arm_id}_link0" />
     </link>
     <link name="${arm_id}_link1">
@@ -60,4 +82,5 @@
         </geometry>
       </collision>
+      <xacro:panda-inertials name="${arm_id}_link1" />
     </link>
     <joint name="${arm_id}_joint1" type="revolute">
@@ -93,4 +116,5 @@
         </geometry>
       </collision>
+      <xacro:panda-inertials name="${arm_id}_link2" />
     </link>
     <joint name="${arm_id}_joint2" type="revolute">
@@ -126,4 +150,5 @@
         </geometry>
       </collision>
+      <xacro:panda-inertials name="${arm_id}_link3" />
     </link>
     <joint name="${arm_id}_joint3" type="revolute">
@@ -159,4 +184,5 @@
         </geometry>
       </collision>
+      <xacro:panda-inertials name="${arm_id}_link4" />
     </link>
     <joint name="${arm_id}_joint4" type="revolute">
@@ -210,4 +236,5 @@
         </geometry>
       </collision>
+      <xacro:panda-inertials name="${arm_id}_link5" />
     </link>
     <joint name="${arm_id}_joint5" type="revolute">
@@ -243,4 +270,5 @@
         </geometry>
       </collision>
+      <xacro:panda-inertials name="${arm_id}_link6" />
     </link>
     <joint name="${arm_id}_joint6" type="revolute">
@@ -276,4 +304,5 @@
         </geometry>
       </collision>
+      <xacro:panda-inertials name="${arm_id}_link7" />
     </link>
     <joint name="${arm_id}_joint7" type="revolute">

File: franka_description/robots/sim/panda_arm_sim.urdf.xacro (robot description, xacro)
@@ -5,8 +5,8 @@
   <xacro:arg name="initial_positions" default="0.0 ${-pi/4} 0.0 ${-3*pi/4} 0.0 ${pi/2} ${pi/4}"/> <!-- initial joint positions of the robot-->
   <xacro:include filename="$(find franka_description)/robots/common/panda_arm.xacro"/>
-  <xacro:panda_arm arm_id="$(arg arm_id)" safety_distance="0.03"/>
+  <xacro:panda_arm arm_id="$(arg arm_id)" safety_distance="0.03" inertials="${xacro.load_yaml('$(find franka_description)/robots/inertials.yaml')}"/>
   <xacro:if value="$(arg hand)">
     <xacro:include filename="$(find franka_description)/robots/common/hand.xacro"/>
-    <xacro:hand ns="$(arg arm_id)" rpy="0 0 ${-pi/4}" connected_to="$(arg arm_id)_link8" safety_distance="0.03"/>
+    <xacro:hand ns="$(arg arm_id)" rpy="0 0 ${-pi/4}" connected_to="$(arg arm_id)_link8" safety_distance="0.03" ee_inertials="${xacro.load_yaml('$(find franka_description)/robots/ee_inertials.yaml')}"/>
   </xacro:if>
   <xacro:include filename="$(find franka_description)/robots/sim/panda_arm_sim.ros2_control.xacro"/>
